Commit message: Suspension mounts added.

File: robot/sawppy.urdf.xacro (robot description, xacro)
@@ -7,4 +7,9 @@
     <xacro:property name="chassis_width" value="0.270"/>
     <xacro:property name="corner_height" value="0.080"/>
+    <!-- Distance between horizontal hole and upper and lower profile's central
+    axes. Distance between the central hole and both axes are different -->
+    <xacro:property name="suspension_mount_upper_dist" value="0.035"/>
+    <xacro:property name="suspension_mount_lower_dist" value="0.045"/>
+    <xacro:property name="suspension_mount_offset_x" value="0.073"/>
     <!-- INCLUDES -->
     <xacro:include filename="$(find sawppy_description)/urdf/common_properties.xacro"/>

File: urdf/body.urdf.xacro (robot description, xacro)
@@ -3,4 +3,5 @@
     <xacro:include filename="$(find sawppy_description)/urdf/profile.urdf.xacro"/>
     <xacro:include filename="$(find sawppy_description)/urdf/body_corner.urdf.xacro"/>
+    <xacro:include filename="$(find sawppy_description)/urdf/suspension_mount.urdf.xacro"/>
     <xacro:macro name="body">
         <!-- ELEMENTS -->
@@ -70,3 +71,12 @@
         <origin xyz="-${chassis_lenght/2} ${chassis_width/2} ${bottom_plate_height + corner_height/2 + profile_width/2}" rpy="0.0 0.0 -${PI/2}"/>
     </xacro:body_corner>
+    <!-- SUSPENSION MOUNTS -->
+    <!-- SUSPENSION MOUNT - RIGHT -->
+    <xacro:suspension_mount suffix="r" parent="base_link">
+        <origin xyz="${suspension_mount_offset_x} -${chassis_width/2} ${bottom_plate_height + suspension_mount_lower_dist + profile_width/2}" rpy="0.0 0.0 0.0"/>
+    </xacro:suspension_mount>
+    <!-- SUSPENSION MOUNT - LEFT -->
+    <xacro:suspension_mount suffix="l" parent="base_link">
+        <origin xyz="${suspension_mount_offset_x} ${chassis_width/2} ${bottom_plate_height + suspension_mount_lower_dist + profile_width/2}" rpy="0.0 0.0 0.0"/>
+    </xacro:suspension_mount>
 </robot>

Commit message: Differential mounts done.

File: robot/sawppy.urdf.xacro (robot description, xacro)
@@ -6,5 +6,7 @@
     <xacro:property name="chassis_lenght" value="0.410"/>
     <xacro:property name="chassis_width" value="0.270"/>
-    <xacro:property name="corner_height" value="0.080"/>
+    <xacro:property name="corner_height" value="0.080"/> <!-- Remove -->
+    <xacro:property name="chassis_height" value="0.080"/>
+    <xacro:property name="differential_offset_x" value="0.00"/>
     <!-- Distance between horizontal hole and upper and lower profile's central
     axes. Distance between the central hole and both axes are different -->

File: urdf/body.urdf.xacro (robot description, xacro)
@@ -4,4 +4,6 @@
     <xacro:include filename="$(find sawppy_description)/urdf/body_corner.urdf.xacro"/>
     <xacro:include filename="$(find sawppy_description)/urdf/suspension_mount.urdf.xacro"/>
+    <xacro:include filename="$(find sawppy_description)/urdf/battery_tray.urdf.xacro"/>
+    <xacro:include filename="$(find sawppy_description)/urdf/differential.urdf.xacro"/>
     <xacro:macro name="body">
         <!-- ELEMENTS -->
@@ -80,3 +82,10 @@
         <origin xyz="${suspension_mount_offset_x} ${chassis_width/2} ${bottom_plate_height + suspension_mount_lower_dist + profile_width/2}" rpy="0.0 0.0 0.0"/>
     </xacro:suspension_mount>
+    <!-- BATTERY TRAY -->
+    <xacro:battery_tray parent="base_link">
+        <origin xyz="-${chassis_lenght/2} 0.0 ${bottom_plate_height + profile_width/2}" rpy="0.0 0.0 0.0"/>
+    </xacro:battery_tray>
+    <!-- DIFFERENTIAL -->
+    <xacro:differential parent="base_link" offset_x="0.0">
+    </xacro:differential>
 </robot>

Commit message: Differential implemented in a new macro with its own base frame, differential_link.

File: robot/sawppy.urdf.xacro (robot description, xacro)
@@ -8,5 +8,5 @@
     <xacro:property name="corner_height" value="0.080"/> <!-- Remove -->
     <xacro:property name="chassis_height" value="0.080"/>
-    <xacro:property name="differential_offset_x" value="0.00"/>
+    <xacro:property name="differential_offset_x" value="-0.015"/>
     <!-- Distance between horizontal hole and upper and lower profile's central
     axes. Distance between the central hole and both axes are different -->

File: urdf/body.urdf.xacro (robot description, xacro)
@@ -73,5 +73,7 @@
         <origin xyz="-${chassis_lenght/2} ${chassis_width/2} ${bottom_plate_height + corner_height/2 + profile_width/2}" rpy="0.0 0.0 -${PI/2}"/>
     </xacro:body_corner>
+    <!--                   -->
     <!-- SUSPENSION MOUNTS -->
+    <!--                   -->
     <!-- SUSPENSION MOUNT - RIGHT -->
     <xacro:suspension_mount suffix="r" parent="base_link">
@@ -86,6 +88,10 @@
         <origin xyz="-${chassis_lenght/2} 0.0 ${bottom_plate_height + profile_width/2}" rpy="0.0 0.0 0.0"/>
     </xacro:battery_tray>
+    <!--              -->
     <!-- DIFFERENTIAL -->
-    <xacro:differential parent="base_link" offset_x="0.0">
+    <!--              -->
+    <!-- xacro:differential parent="base_link" offset_x="0.0" -->
+    <xacro:differential parent="base_link">
+        <origin xyz="${differential_offset_x} 0.0 ${bottom_plate_height + chassis_height + profile_width/2}" rpy="0.0 0.0 0.0"/>
     </xacro:differential>
 </robot>

File: urdf/common_properties.xacro (robot description, xacro)
@@ -6,4 +6,7 @@
     <!-- PARAMETERS -->
     <!-- COLORS -->
+    <material name="black">
+        <color rgba="0.0 0.0 0.0 1.0"/>
+    </material>
     <material name="glass">
         <color rgba="0.7 0.7 0.7 0.5"/>
@@ -15,6 +18,6 @@
         <color rgba="0.95 0.95 0.95 1.0"/>
     </material>
-    <material name="black">
-        <color rgba="0.0 0.0 0.0 1.0"/>
+    <material name="steel">
+        <color rgba="0.3 0.3 0.3 1.0"/>
     </material>
 </robot>

File: urdf/differential.urdf.xacro (robot description, xacro)
@@ -1,10 +1,25 @@
 <?xml version="1.0"?>
 <robot xmlns:xacro="http://ros.org/wiki.xacro">
-    <xacro:macro name="differential" params="parent offset_x">
-        <!-- Right differential mount -->
-        <joint name="${parent}_to_differential_mount_r" type="fixed">
+    <xacro:property name="rod_offset_z" value="0.0257"/>
+    <xacro:macro name="differential" params="parent *origin">
+        <!-- BASE REFERENCE FRAME FOR THE DIFFERENTIAL -->
+        <joint name="differential_mount" type="fixed">
             <parent link="${parent}"/>
+            <child link="differential_link"/>
+            <xacro:insert_block name="origin"/>
+        </joint>
+        <link name="differential_link">
+            <visual>
+                <origin xyz="0.0 0.0 0.0" rpy="0.0 0.0 0.0"/>
+                <geometry>
+                    <box size="0.0001 0.0001 0.0001"/>
+                </geometry>
+            </visual>
+        </link>
+        <!-- RIGHT DIFFERENTIAL MOUNT -->
+        <joint name="differential_to_differential_mount_r" type="fixed">
+            <parent link="differential_link"/>
             <child link="differential_mount_r"/>
-            <origin xyz="${offset_x} -${chassis_width/2} ${bottom_plate_height + chassis_height + profile_width/2}" rpy="0.0 0.0 0.0"/>
+            <origin xyz="0.0 -${chassis_width/2} 0.0" rpy="0.0 0.0 0.0"/>
         </joint>
         <link name="differential_mount_r">
@@ -17,9 +32,9 @@
             </visual>
         </link>
-        <!-- Left differential mount-->
-        <joint name="${parent}_to_differential_mount_l" type="fixed">
-            <parent link="${parent}"/>
+        <!-- LEFT DIFFERENTIAL MOUNT -->
+        <joint name="differential_to_differential_mount_l" type="fixed">
+            <parent link="differential_link"/>
             <child link="differential_mount_l"/>
-            <origin xyz="${offset_x} ${chassis_width/2} ${bottom_plate_height + chassis_height + profile_width/2}" rpy="0.0 0.0 0.0"/>
+            <origin xyz="0.0 ${chassis_width/2} 0.0" rpy="0.0 0.0 0.0"/>
         </joint>
         <link name="differential_mount_l">
@@ -33,18 +48,81 @@
         </link>
         <!-- Differential profile -->
-        <joint name="${parent}_to_differential_mount_l" type="fixed">
-            <parent link="${parent}"/>
-            <child link="differential_mount_l"/>
-            <origin xyz="${offset_x} ${chassis_width/2} ${bottom_plate_height + chassis_height + profile_width/2}" rpy="0.0 0.0 0.0"/>
+        <xacro:profile suffix="diff" parent="differential_link" length="245">
+            <origin xyz="0.0 0.0 0.0" rpy="0.0 0.0 ${PI/2}"/>
+        </xacro:profile>
+        <!-- DIFFERENTIAL SUPPORT -->
+        <joint name="differential_to_support_lower" type="fixed">
+            <parent link="differential_link"/>
+            <child link="differential_support_lower"/>
+            <origin xyz="0.0 0.0 0.0" rpy="0.0 0.0 0.0"/>
         </joint>
-        <link name="differential_mount_l">
+        <link name="differential_support_lower">
             <visual>
                 <origin xyz="0.0 0.0 0.0" rpy="0.0 0.0 ${PI/2}"/>
                 <geometry>
-                    <mesh filename="package://sawppy_description/meshes/stl/differential_mount_left.stl" scale="${SCALE}"/>
+                    <mesh filename="package://sawppy_description/meshes/stl/differential_support_lower.stl" scale="${SCALE}"/>
                 </geometry>
                 <material name="plastic"/>
             </visual>
         </link>
+        <joint name="differential_to_support_upper" type="fixed">
+            <parent link="differential_link"/>
+            <child link="differential_support_upper"/>
+            <origin xyz="0.0 0.0 0.0" rpy="0.0 0.0 0.0"/>
+        </joint>
+        <link name="differential_support_upper">
+            <visual>
+                <origin xyz="0.0 0.0 ${0.0254-profile_width/2}" rpy="0.0 0.0 ${PI/2}"/>
+                <geometry>
+                    <mesh filename="package://sawppy_description/meshes/stl/differential_support_upper.stl" scale="${SCALE}"/>
+                </geometry>
+                <material name="plastic"/>
+            </visual>
+        </link>
+        <!-- ROD SUPPORT -->
+        <joint name="differential_to_rod_support" type="fixed">
+            <parent link="differential_link"/>
+            <child link="differential_rod_support"/>
+            <origin xyz="0.0 0.0 0.0" rpy="0.0 0.0 0.0"/>
+        </joint>
+        <link name="differential_rod_support">
+            <visual>
+                <origin xyz="0.0 0.0 ${rod_offset_z}" rpy="0.0 0.0 ${PI/2}"/>
+                <geometry>
+                    <mesh filename="package://sawppy_description/meshes/stl/differential_rod_support.stl" scale="${SCALE}"/>
+                </geometry>
+                <material name="plastic"/>
+            </visual>
+        </link>
+        <!-- DIFFERENTIAL BRACE -->
+        <joint name="differential_to_brace" type="fixed">
+            <parent link="differential_link"/>
+            <child link="differential_brace"/>
+            <origin xyz="0.0 0.0 0.0" rpy="0.0 0.0 0.0"/>
+        </joint>
+        <link name="differential_brace">
+            <visual>
+                <origin xyz="0.0 0.0 ${rod_offset_z}" rpy="0.0 0.0 ${PI/2}"/>
+                <geometry>
+                    <mesh filename="package://sawppy_description/meshes/stl/differential_brace.stl" scale="${SCALE}"/>
+                </geometry>
+                <material name="plastic"/>
+            </visual>
+        </link>
+        <!-- DIFFERENTIAL ROD -->
+        <joint name="differential_to_rod" type="fixed">
+            <parent link="differential_link"/>
+            <child link="differential_rod"/>
+            <origin xyz="0.0 0.0 0.0" rpy="0.0 0.0 0.0"/>
+        </joint>
+        <link name="differential_rod">
+            <visual>
+                <origin xyz="0.0 0.0 ${rod_offset_z}" rpy="0.0 0.0 ${PI/2}"/>
+                <geometry>
+                    <mesh filename="package://sawppy_description/meshes/stl/differential_rod.stl" scale="${SCALE}"/>
+                </geometry>
+                <material name="steel"/>
+            </visual>
+        </link>
     </xacro:macro>
 </robot>

Commit message: Rocker joint and first two Rocker-Bogie profiles added.

File: robot/sawppy.urdf.xacro (robot description, xacro)
@@ -14,8 +14,15 @@
     <xacro:property name="suspension_mount_lower_dist" value="0.045"/>
     <xacro:property name="suspension_mount_offset_x" value="0.073"/>
+    <xacro:property name="suspension_mount_width" value="0.040"/>
     <!-- INCLUDES -->
     <xacro:include filename="$(find sawppy_description)/urdf/common_properties.xacro"/>
     <xacro:include filename="$(find sawppy_description)/urdf/body.urdf.xacro"/>
+    <xacro:include filename="$(find sawppy_description)/urdf/rocker_bogie_left.urdf.xacro"/>
     <!-- BODY CHASSIS -->
     <xacro:body/>
+    <!-- ROCKER-BOGIE - RIGHT -->
+    <!-- ROCKER-BOGIE - LEFT -->
+    <xacro:rocker_bogie_left parent="suspension_left">
+        <origin xyz="0.0 ${suspension_mount_width/2 + 0.001} 0.0" rpy="0.0 0.0 0.0"/>
+    </xacro:rocker_bogie_left>
 </robot>

File: urdf/body.urdf.xacro (robot description, xacro)
@@ -77,9 +77,9 @@
     <!--                   -->
     <!-- SUSPENSION MOUNT - RIGHT -->
-    <xacro:suspension_mount suffix="r" parent="base_link">
+    <xacro:suspension_mount suffix="right" parent="base_link">
         <origin xyz="${suspension_mount_offset_x} -${chassis_width/2} ${bottom_plate_height + suspension_mount_lower_dist + profile_width/2}" rpy="0.0 0.0 0.0"/>
     </xacro:suspension_mount>
     <!-- SUSPENSION MOUNT - LEFT -->
-    <xacro:suspension_mount suffix="l" parent="base_link">
+    <xacro:suspension_mount suffix="left" parent="base_link">
         <origin xyz="${suspension_mount_offset_x} ${chassis_width/2} ${bottom_plate_height + suspension_mount_lower_dist + profile_width/2}" rpy="0.0 0.0 0.0"/>
     </xacro:suspension_mount>
@@ -91,5 +91,4 @@
     <!-- DIFFERENTIAL -->
     <!--              -->
-    <!-- xacro:differential parent="base_link" offset_x="0.0" -->
     <xacro:differential parent="base_link">
         <origin xyz="${differential_offset_x} 0.0 ${bottom_plate_height + chassis_height + profile_width/2}" rpy="0.0 0.0 0.0"/>

File: urdf/differential.urdf.xacro (robot description, xacro)
@@ -1,3 +1,7 @@
 <?xml version="1.0"?>
+<!--
+[ ] CHANGE FIXED JOINTS TO THE CORRECT TYPE.
+[ ] MODIFY PARENT LINKS TO MAKE EACH LINK DEPEND ON THE ONE THAT SUPPORTS IT
+ -->
 <robot xmlns:xacro="http://ros.org/wiki.xacro">
     <xacro:property name="rod_offset_z" value="0.0257"/>

Commit message: Refactoring. Interior bogie joint added.

File: robot/sawppy.urdf.xacro (robot description, xacro)
@@ -9,20 +9,25 @@
     <xacro:property name="chassis_height" value="0.080"/>
     <xacro:property name="differential_offset_x" value="-0.015"/>
-    <!-- Distance between horizontal hole and upper and lower profile's central
-    axes. Distance between the central hole and both axes are different -->
-    <xacro:property name="suspension_mount_upper_dist" value="0.035"/>
-    <xacro:property name="suspension_mount_lower_dist" value="0.045"/>
-    <xacro:property name="suspension_mount_offset_x" value="0.073"/>
-    <xacro:property name="suspension_mount_width" value="0.040"/>
     <!-- INCLUDES -->
     <xacro:include filename="$(find sawppy_description)/urdf/common_properties.xacro"/>
     <xacro:include filename="$(find sawppy_description)/urdf/body.urdf.xacro"/>
-    <xacro:include filename="$(find sawppy_description)/urdf/rocker_bogie_left.urdf.xacro"/>
+    <xacro:include filename="$(find sawppy_description)/urdf/rocker_bogie.urdf.xacro"/>
     <!-- BODY CHASSIS -->
     <xacro:body/>
     <!-- ROCKER-BOGIE - RIGHT -->
+    <xacro:rocker_bogie suffix="right" parent="base_link" reflect="1"/>
+        <!--
+        <origin xyz="0.0 ${suspension_mount_width/2 + 0.001} 0.0" rpy="0.0 0.0 0.0"/>
+        -->
+        <!--
+        <origin xyz="${suspension_mount_offset_x} -${chassis_width/2} ${bottom_plate_height + suspension_mount_lower_dist + profile_width/2}" rpy="0.0 0.0 0.0"/>
+    </xacro:rocker_bogie>
+        -->
     <!-- ROCKER-BOGIE - LEFT -->
-    <xacro:rocker_bogie_left parent="suspension_left">
-        <origin xyz="0.0 ${suspension_mount_width/2 + 0.001} 0.0" rpy="0.0 0.0 0.0"/>
-    </xacro:rocker_bogie_left>
+    <xacro:rocker_bogie suffix="left" parent="base_link" reflect="-1"/>
+    <!--
+    <xacro:rocker_bogie suffix="left" parent="base_link" reflect="-1">
+        <origin xyz="${suspension_mount_offset_x} ${chassis_width/2} ${bottom_plate_height + suspension_mount_lower_dist + profile_width/2}" rpy="0.0 0.0 0.0"/>
+    </xacro:rocker_bogie>
+    -->
 </robot>

File: urdf/body.urdf.xacro (robot description, xacro)
@@ -77,11 +77,15 @@
     <!--                   -->
     <!-- SUSPENSION MOUNT - RIGHT -->
+    <!--
     <xacro:suspension_mount suffix="right" parent="base_link">
         <origin xyz="${suspension_mount_offset_x} -${chassis_width/2} ${bottom_plate_height + suspension_mount_lower_dist + profile_width/2}" rpy="0.0 0.0 0.0"/>
     </xacro:suspension_mount>
+    -->
     <!-- SUSPENSION MOUNT - LEFT -->
+    <!--
     <xacro:suspension_mount suffix="left" parent="base_link">
         <origin xyz="${suspension_mount_offset_x} ${chassis_width/2} ${bottom_plate_height + suspension_mount_lower_dist + profile_width/2}" rpy="0.0 0.0 0.0"/>
     </xacro:suspension_mount>
+    -->
     <!-- BATTERY TRAY -->
     <xacro:battery_tray parent="base_link">

File: urdf/suspension_mount.urdf.xacro (robot description, xacro)
@@ -1,13 +1,19 @@
 <?xml version="1.0"?>
 <robot xmlns:xacro="http://ros.org/wiki.xacro">
+    <!-- Distance between horizontal hole and upper and lower profile's central
+    axes. Distance between the central hole and both axes are different -->
+    <xacro:property name="suspension_mount_upper_dist" value="0.035"/>
+    <xacro:property name="suspension_mount_lower_dist" value="0.045"/>
+    <xacro:property name="suspension_mount_offset_x" value="0.073"/>
+    <xacro:property name="suspension_mount_width" value="0.040"/>
     <xacro:macro name="suspension_mount" params="suffix parent *origin">
         <joint name="${parent}_to_${suffix}_suspension" type="fixed">
             <parent link="${parent}"/>
             <child link="suspension_${suffix}"/>
-            <xacro:insert_block name="origin"/>
+        <origin xyz="${suspension_mount_offset_x} ${-reflect*chassis_width/2} ${bottom_plate_height + suspension_mount_lower_dist + profile_width/2}" rpy="0.0 0.0 0.0"/>
         </joint>
         <link name="suspension_${suffix}">
             <visual>
-                <origin xyz="0.0 0.0 0.0" rpy="0.0 0.0 ${PI/2}"/>
+                <origin xyz="0.0 0.0 0.0" rpy="0.0 0.0 ${-reflect*PI/2}"/>
                 <geometry>
                     <mesh filename="package://sawppy_description/meshes/stl/suspension_mount.stl" scale="${SCALE}"/>
